File: Wheelmod_rs485.sch (EAGLE design)
At the start: 52 parts, among them IC1 SN75176BPSR, SW1 RST_SW, SW2 HWB_SW, U1 ATMEGA8U2AU, U2 SI8441IS1, U3 MC33887-HSOP, U4 NFET-SOIC8, U5 LDO, X1 MINI-USB, X2 MICROMATCH-4, X3 ENC, X4 MICROMATCH-4, X5 LOGIC_IN, Y1 SMDRESONATOR

Commit message: Added fixes to Tiina's version
Parts:
- removed IC1: SN75176BPSR, rs485DRIVER:SN75176BPSR
- removed SW1: RST_SW, Erik:SMD-TACT-3.9X2.9
- removed SW2: HWB_SW, Erik:SMD-TACT-3.9X2.9
- removed X2: MICROMATCH-4, con-amp-micromatch:MICROMATCH-4
- added R9: 120, rcl:R-EU_R0603
- added S1: HWB, kommunikatsioonimoodul:ADTSM3
- added S2: RESET, kommunikatsioonimoodul:ADTSM3
- added U$1: SN65HVF76DGS, rs485:SN65HVF76DGS
- added X6: R485-IO, con-amp-micromatch:MICROMATCH-6
Connections:
- removed net N$32: F1.1, X2-2.S
- new net N$33: F1.1, X6-1.S
- new net RE: U$1.RE, U1.PD5
- new net Y: R9.1, U$1.Y, X6-6.S
- new net Z: R9.2, U$1.Z, X6-5.S
- net A: now also R5.2, U$1.A, X6-3.S; no longer IC1.A, R5.1, X2-3.S
- net B: now also R5.1, U$1.B, X6-4.S; no longer IC1.B, R5.2, X2-4.S
- net DE: now also U$1.DE; no longer IC1.DE, IC1.RE
- net GND: now also S1.1, S2.1, U$1.GND, X6-2.S; no longer IC1.GND, SW1.1, SW2.2, X2-1.S
- net N$10: now also S2.2; no longer SW1.2
- net N$2: now also S1.2; no longer SW2.1
- net RX: now also U$1.R; no longer IC1.R
- net TX: now also U$1.D; no longer IC1.D
- net VCC: now also U$1.VCC; no longer IC1.VCC
Other:
- note added: "wheelmod v0.8"
- note removed: "wheelmod v0.7"
- moved on the sheet: C14, C15, C3, C6, C7, C8, D1, F1, F3, JP2, LED4, R13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
